File: hw/flipdot-driver/flipdot-driver.sch (KiCad schematic (older format))
At the start: 93 parts, among them J1 DISPLAY, J2 NRF_CON, J3 Prog, J4 I2C, J5 USART, J6 USB, J7 USB_B_Micro, J8 RST, J9 MAIN_Power, Q1 MMBTA64, Q10 MMBTA64, Q11 MMBTA64, Q12 MMBTA64, Q13 MMBTA64, Q14 MMBTA64, Q15 Q_NMOS_GSD, Q16 Q_NMOS_GSD, Q17 Q_NMOS_GSD, Q18 Q_NMOS_GSD, Q2 MMBTA64, Q3 MMBTA64, Q4 MMBTA64, Q5 MMBTA64, Q6 MMBTA64, Q7 MMBTA64, Q8 MMBTA64, Q9 MMBTA64, U1 AT25xxx, U2 ULN2003A, U3 USBLC6-2SC6, U4 AZ1117-3.3, U5 ULN2003A, U6 stm32_STM32F103C(8-B)Tx, U7 74HC595, U8 AX5201, U9 74HC595, Y1 32768, Y2 8MHz/20pF

Commit message: Placed labels, NRF connector mirrored.
Parts:
- added H1, H2: MountingHole_Pad, MountingHole:MountingHole_3.2mm_M3_DIN965_Pad, symbol Mechanical:MountingHole_Pad
- C10, C11, C12, C13, C14, C15, C17, C18, C19, C20, C22, C5, C6, C7, C8, C9: symbol flipdot-driver-rescue:C-controller-cache-flipdot-driver-rescue -> flipdot-driver-rescue:C-controller-cache-flipdot-driver-rescue-flipdot-driver-rescue
- C16, C21, C23: symbol flipdot-driver-rescue:CP-controller-cache-flipdot-driver-rescue -> flipdot-driver-rescue:CP-controller-cache-flipdot-driver-rescue-flipdot-driver-rescue
- D2, D6: symbol flipdot-driver-rescue:D_Schottky-controller-cache-flipdot-driver-rescue -> flipdot-driver-rescue:D_Schottky-controller-cache-flipdot-driver-rescue-flipdot-driver-rescue
- D7, D8: symbol flipdot-driver-rescue:LED-controller-cache-flipdot-driver-rescue -> flipdot-driver-rescue:LED-controller-cache-flipdot-driver-rescue-flipdot-driver-rescue
- L2: symbol flipdot-driver-rescue:L-controller-cache-flipdot-driver-rescue -> flipdot-driver-rescue:L-controller-cache-flipdot-driver-rescue-flipdot-driver-rescue
- R11, R12: symbol controller-cache:R -> flipdot-driver-rescue:R-controller-cache
- R36: symbol flipdot-driver-rescue:R-controller-cache-flipdot-driver-rescue -> flipdot-driver-rescue:R-controller-cache-flipdot-driver-rescue-flipdot-driver-rescue
- U6: symbol flipdot-driver-rescue:stm32_STM32F103C(8-B)Tx-STM32_converter-cache-flipdot-driver-rescue -> flipdot-driver-rescue:stm32_STM32F103C(8-B)Tx-STM32_converter-cache-flipdot-driver-rescue-flipdot-driver-rescue
- U8: symbol flipdot-driver-rescue:AX5201-LCSC -> flipdot-driver-rescue:AX5201-LCSC-flipdot-driver-rescue
Connections:
- net GND: now also H1.1, H2.1
Changed lines of the file:
@@
 $EndComp
 $Comp
-L flipdot-driver-rescue:C-controller-cache-flipdot-driver-rescue C14
+L flipdot-driver-rescue:C-controller-cache-flipdot-driver-rescue-flipdot-driver-rescue C14
 U 1 1 5C81535A
 P 15050 4500
@@
 $EndComp
 $Comp
-L flipdot-driver-rescue:C-controller-cache-flipdot-driver-rescue C15
+L flipdot-driver-rescue:C-controller-cache-flipdot-driver-rescue-flipdot-driver-rescue C15
 U 1 1 5C815450
 P 15400 4500
@@
 NRF_IRQ
 $Comp
-L flipdot-driver-rescue:C-controller-cache-flipdot-driver-rescue C5
+L flipdot-driver-rescue:C-controller-cache-flipdot-driver-rescue-flipdot-driver-rescue C5
 U 1 1 5C98C3EA
 P 7700 6700
@@
 $EndComp
 $Comp
-L flipdot-driver-rescue:C-controller-cache-flipdot-driver-rescue C6
+L flipdot-driver-rescue:C-controller-cache-flipdot-driver-rescue-flipdot-driver-rescue C6
 U 1 1 5C98C4BA
 P 8000 6700
@@
 $EndComp
 $Comp
-L flipdot-driver-rescue:C-controller-cache-flipdot-driver-rescue C7
+L flipdot-driver-rescue:C-controller-cache-flipdot-driver-rescue-flipdot-driver-rescue C7
 U 1 1 5C98C550
 P 8300 6700
@@
 $EndComp
 $Comp
-L flipdot-driver-rescue:C-controller-cache-flipdot-driver-rescue C8
+L flipdot-driver-rescue:C-controller-cache-flipdot-driver-rescue-flipdot-driver-rescue C8
 U 1 1 5C98C5EC
 P 8600 6700
@@
 $EndComp
 $Comp
-L flipdot-driver-rescue:C-controller-cache-flipdot-driver-rescue C9
+L flipdot-driver-rescue:C-controller-cache-flipdot-driver-rescue-flipdot-driver-rescue C9
 U 1 1 5CA62C8B
 P 6550 1150
@@
 $EndComp
 $Comp
-L flipdot-driver-rescue:C-controller-cache-flipdot-driver-rescue C11
+L flipdot-driver-rescue:C-controller-cache-flipdot-driver-rescue-flipdot-driver-rescue C11
 U 1 1 5CA62D35
 P 7600 1150
@@
 $EndComp
 $Comp
-L flipdot-driver-rescue:C-controller-cache-flipdot-driver-rescue C12
+L flipdot-driver-rescue:C-controller-cache-flipdot-driver-rescue-flipdot-driver-rescue C12
 U 1 1 5CC51283
 P 7600 4250
@@
 $EndComp
 $Comp
-L flipdot-driver-rescue:C-controller-cache-flipdot-driver-rescue C13
+L flipdot-driver-rescue:C-controller-cache-flipdot-driver-rescue-flipdot-driver-rescue C13
 U 1 1 5CC5134B
 P 7900 4250
@@
 	7150 6200 7150 6100
 $Comp
-L flipdot-driver-rescue:C-controller-cache-flipdot-driver-rescue C10
+L flipdot-driver-rescue:C-controller-cache-flipdot-driver-rescue-flipdot-driver-rescue C10
 U 1 1 5D06CD87
 P 7350 6350
@@
 USART_RX
 $Comp
-L flipdot-driver-rescue:D_Schottky-controller-cache-flipdot-driver-rescue D6
+L flipdot-driver-rescue:D_Schottky-controller-cache-flipdot-driver-rescue-flipdot-driver-rescue D6
 U 1 1 5C783BF6
 P 8700 1150
@@
 $EndComp
 $Comp
-L flipdot-driver-rescue:R-controller-cache-flipdot-driver-rescue R36
+L flipdot-driver-rescue:R-controller-cache-flipdot-driver-rescue-flipdot-driver-rescue R36
 U 1 1 5C29AE4A
 P 7200 2150
@@
 	15000 2350 15500 2350
 $Comp
-L flipdot-driver-rescue:stm32_STM32F103C(8-B)Tx-STM32_converter-cache-flipdot-driver-rescue U6
+L flipdot-driver-rescue:stm32_STM32F103C(8-B)Tx-STM32_converter-cache-flipdot-driver-rescue-flipdot-driver-rescue U6
 U 1 1 5C4F9114
 P 11600 4150
@@
 $EndComp
 $Comp
-L flipdot-driver-rescue:LED-controller-cache-flipdot-driver-rescue D7
+L flipdot-driver-rescue:LED-controller-cache-flipdot-driver-rescue-flipdot-driver-rescue D7
 U 1 1 5DEBAEF3
 P 5650 4350
@@
 $EndComp
 $Comp
-L flipdot-driver-rescue:LED-controller-cache-flipdot-driver-rescue D8
+L flipdot-driver-rescue:LED-controller-cache-flipdot-driver-rescue-flipdot-driver-rescue D8
 U 1 1 5DF44183
 P 6400 4350
@@
 $EndComp
 $Comp
-L flipdot-driver-rescue:CP-controller-cache-flipdot-driver-rescue C16
+L flipdot-driver-rescue:CP-controller-cache-flipdot-driver-rescue-flipdot-driver-rescue C16
 U 1 1 5CF6C5C2
 P 700 2850
@@
 $EndComp
 $Comp
-L flipdot-driver-rescue:C-controller-cache-flipdot-driver-rescue C17
+L flipdot-driver-rescue:C-controller-cache-flipdot-driver-rescue-flipdot-driver-rescue C17
 U 1 1 5CF6CCDF
 P 1050 3000
@@
 $EndComp
 $Comp
-L flipdot-driver-rescue:L-controller-cache-flipdot-driver-rescue L2
+L flipdot-driver-rescue:L-controller-cache-flipdot-driver-rescue-flipdot-driver-rescue L2
 U 1 1 5CF6D440
 P 2600 2350
@@
 $EndComp
 $Comp
-L flipdot-driver-rescue:D_Schottky-controller-cache-flipdot-driver-rescue D2
+L flipdot-driver-rescue:D_Schottky-controller-cache-flipdot-driver-rescue-flipdot-driver-rescue D2
 U 1 1 5CF6DC84
 P 3400 2350
@@
 $EndComp
 $Comp
-L flipdot-driver-rescue:C-controller-cache-flipdot-driver-rescue C20
+L flipdot-driver-rescue:C-controller-cache-flipdot-driver-rescue-flipdot-driver-rescue C20
 U 1 1 5CF6F069
 P 4050 2800
@@
 $EndComp
 $Comp
-L flipdot-driver-rescue:CP-controller-cache-flipdot-driver-rescue C21
+L flipdot-driver-rescue:CP-controller-cache-flipdot-driver-rescue-flipdot-driver-rescue C21
 U 1 1 5CF6F72F
 P 4400 2800
@@
 24V_EN
 $Comp
-L flipdot-driver-rescue:C-controller-cache-flipdot-driver-rescue C19
+L flipdot-driver-rescue:C-controller-cache-flipdot-driver-rescue-flipdot-driver-rescue C19
 U 1 1 5CF703D9
 P 1950 3250
@@
 	800  2550 1050 2550
 $Comp
-L flipdot-driver-rescue:C-controller-cache-flipdot-driver-rescue C18
+L flipdot-driver-rescue:C-controller-cache-flipdot-driver-rescue-flipdot-driver-rescue C18
 U 1 1 5D79E9FF
 P 1350 2850
@@
 Connection ~ 1650 2850
 $Comp
-L flipdot-driver-rescue:AX5201-LCSC U8
+L flipdot-driver-rescue:AX5201-LCSC-flipdot-driver-rescue U8
 U 1 1 5DB4EC83
 P 2600 2950
@@
 USB2_N
 $Comp
-L flipdot-driver-rescue:C-controller-cache-flipdot-driver-rescue C22
+L flipdot-driver-rescue:C-controller-cache-flipdot-driver-rescue-flipdot-driver-rescue C22
 U 1 1 5D0FB237
 P 900 6900
@@
 	900  7050 900  7150
 $Comp
-L controller-cache:R R11
+L flipdot-driver-rescue:R-controller-cache R11
 U 1 1 5D210FC0
 P 4300 5600
@@
 $EndComp
 $Comp
-L controller-cache:R R12
+L flipdot-driver-rescue:R-controller-cache R12
 U 1 1 5D2115E1
 P 4550 5700
@@
 	3700 5700 4150 5700
 $Comp
-L flipdot-driver-rescue:CP-controller-cache-flipdot-driver-rescue C23
+L flipdot-driver-rescue:CP-controller-cache-flipdot-driver-rescue-flipdot-driver-rescue C23
 U 1 1 5D3FC10B
 P 4800 2800
@@
 Wire Wire Line
 	8650 1250 8650 1650
+$Comp
+L Mechanical:MountingHole_Pad H1
+U 1 1 5CF749D3
+P 5350 950
+F 0 "H1" V 5304 1100 50  0000 L CNN
+F 1 "MountingHole_Pad" V 5395 1100 50  0000 L CNN
+F 2 "MountingHole:MountingHole_3.2mm_M3_DIN965_Pad" H 5350 950 50  0001 C CNN
+F 3 "~" H 5350 950 50  0001 C CNN
+	1    5350 950
+	0    1    1    0
+$EndComp
+$Comp
+L Mechanical:MountingHole_Pad H2
+U 1 1 5CF763BF
+P 5350 1200
+F 0 "H2" V 5304 1350 50  0000 L CNN
+F 1 "MountingHole_Pad" V 5395 1350 50  0000 L CNN
+F 2 "MountingHole:MountingHole_3.2mm_M3_DIN965_Pad" H 5350 1200 50  0001 C CNN
+F 3 "~" H 5350 1200 50  0001 C CNN
+	1    5350 1200
+	0    1    1    0
+$EndComp
+$Comp
+L power:GND #PWR0102
+U 1 1 5CF76D90
+P 5150 1750
+F 0 "#PWR0102" H 5150 1500 50  0001 C CNN
+F 1 "GND" H 5155 1577 50  0000 C CNN
+F 2 "" H 5150 1750 50  0001 C CNN
+F 3 "" H 5150 1750 50  0001 C CNN
+	1    5150 1750
+	1    0    0    -1
+$EndComp
+Wire Wire Line
+	5150 950  5250 950
+Wire Wire Line
+	5250 1200 5150 1200
+Connection ~ 5150 1200
+Wire Wire Line
+	5150 1200 5150 950
+Wire Wire Line
+	5150 1200 5150 1750
 $EndSCHEMATC

Commit message: Ready for manufacturing.
Parts:
- added FID1, FID2, FID3: Fiducial, Fiducial:Fiducial_0.75mm_Dia_1.5mm_Outer, symbol Mechanical:Fiducial
- C10, C11, C12, C13, C14, C15, C17, C18, C19, C20, C22, C5, C6, C7, C8, C9: symbol flipdot-driver-rescue:C-controller-cache-flipdot-driver-rescue-flipdot-driver-rescue -> flipdot-driver-rescue:C-controller-cache-flipdot-driver-rescue-flipdot-driver-rescue-flipdot-driver-rescue
- C16, C21, C23: symbol flipdot-driver-rescue:CP-controller-cache-flipdot-driver-rescue-flipdot-driver-rescue -> flipdot-driver-rescue:CP-controller-cache-flipdot-driver-rescue-flipdot-driver-rescue-flipdot-driver-rescue
- D2, D6: symbol flipdot-driver-rescue:D_Schottky-controller-cache-flipdot-driver-rescue-flipdot-driver-rescue -> flipdot-driver-rescue:D_Schottky-controller-cache-flipdot-driver-rescue-flipdot-driver-rescue-flipdot-driver-rescue
- D7, D8: symbol flipdot-driver-rescue:LED-controller-cache-flipdot-driver-rescue-flipdot-driver-rescue -> flipdot-driver-rescue:LED-controller-cache-flipdot-driver-rescue-flipdot-driver-rescue-flipdot-driver-rescue
- L2: symbol flipdot-driver-rescue:L-controller-cache-flipdot-driver-rescue-flipdot-driver-rescue -> flipdot-driver-rescue:L-controller-cache-flipdot-driver-rescue-flipdot-driver-rescue-flipdot-driver-rescue
- R11, R12: symbol flipdot-driver-rescue:R-controller-cache -> flipdot-driver-rescue:R-controller-cache-flipdot-driver-rescue
- R36: symbol flipdot-driver-rescue:R-controller-cache-flipdot-driver-rescue-flipdot-driver-rescue -> flipdot-driver-rescue:R-controller-cache-flipdot-driver-rescue-flipdot-driver-rescue-flipdot-driver-rescue
- U6: symbol flipdot-driver-rescue:stm32_STM32F103C(8-B)Tx-STM32_converter-cache-flipdot-driver-rescue-flipdot-driver-rescue -> flipdot-driver-rescue:stm32_STM32F103C(8-B)Tx-STM32_converter-cache-flipdot-driver-rescue-flipdot-driver-rescue-flipdot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
- U8: symbol flipdot-driver-rescue:AX5201-LCSC-flipdot-driver-rescue -> flipdot-driver-rescue:AX5201-LCSC-flipdot-driver-rescue-flipdot-driver-rescue
Connections:
- net +3V3: now also J2.1 (Pin_1); no longer J2.2 (Pin_2)
- net GND: now also J2.2 (Pin_2); no longer J2.1 (Pin_1)
- net NRF_CE: now also J2.4 (Pin_4); no longer J2.3 (Pin_3)
- net NRF_IRQ: now also J2.7 (Pin_7); no longer J2.8 (Pin_8)
- net NRF_SS: now also J2.3 (Pin_3); no longer J2.4 (Pin_4)
- net SPI_MISO: now also J2.8 (Pin_8); no longer J2.7 (Pin_7)
- net SPI_MOSI: now also J2.5 (Pin_5); no longer J2.6 (Pin_6)
- net SPI_SCK: now also J2.6 (Pin_6); no longer J2.5 (Pin_5)
Changed lines of the file:
@@
 L Connector_Generic:Conn_02x04_Odd_Even J2
 U 1 1 5C6A6837
-P 2000 6100
-F 0 "J2" H 2050 6417 50  0000 C CNN
-F 1 "NRF_CON" H 2050 6326 50  0000 C CNN
-F 2 "Connector_PinSocket_2.54mm:PinSocket_2x04_P2.54mm_Vertical" H 2000 6100 50  0001 C CNN
-F 3 "~" H 2000 6100 50  0001 C CNN
-	1    2000 6100
-	1    0    0    -1
+P 2100 6100
+F 0 "J2" H 2150 6417 50  0000 C CNN
+F 1 "NRF_CON" H 2150 6326 50  0000 C CNN
+F 2 "Connector_PinSocket_2.54mm:PinSocket_2x04_P2.54mm_Vertical" H 2100 6100 50  0001 C CNN
+F 3 "~" H 2100 6100 50  0001 C CNN
+	1    2100 6100
+	-1   0    0    -1
 $EndComp
 Wire Wire Line
@@
 $EndComp
 $Comp
-L flipdot-driver-rescue:C-controller-cache-flipdot-driver-rescue-flipdot-driver-rescue C14
+L flipdot-driver-rescue:C-controller-cache-flipdot-driver-rescue-flipdot-driver-rescue-flipdot-driver-rescue C14
 U 1 1 5C81535A
 P 15050 4500
@@
 $EndComp
 $Comp
-L flipdot-driver-rescue:C-controller-cache-flipdot-driver-rescue-flipdot-driver-rescue C15
+L flipdot-driver-rescue:C-controller-cache-flipdot-driver-rescue-flipdot-driver-rescue-flipdot-driver-rescue C15
 U 1 1 5C815450
 P 15400 4500
@@
 	1300 6050 1300 6000
 Wire Wire Line
-	1300 6000 1800 6000
-Wire Wire Line
 	2300 6000 2700 6000
 Wire Wire Line
 	2700 6000 2700 5950
-Wire Wire Line
-	1800 6100 1450 6100
-Wire Wire Line
-	1800 6200 1450 6200
-Wire Wire Line
-	1800 6300 1450 6300
 Wire Wire Line
 	2300 6100 2700 6100
@@
 NRF_IRQ
 $Comp
-L flipdot-driver-rescue:C-controller-cache-flipdot-driver-rescue-flipdot-driver-rescue C5
+L flipdot-driver-rescue:C-controller-cache-flipdot-driver-rescue-flipdot-driver-rescue-flipdot-driver-rescue C5
 U 1 1 5C98C3EA
 P 7700 6700
@@
 $EndComp
 $Comp
-L flipdot-driver-rescue:C-controller-cache-flipdot-driver-rescue-flipdot-driver-rescue C6
+L flipdot-driver-rescue:C-controller-cache-flipdot-driver-rescue-flipdot-driver-rescue-flipdot-driver-rescue C6
 U 1 1 5C98C4BA
 P 8000 6700
@@
 $EndComp
 $Comp
-L flipdot-driver-rescue:C-controller-cache-flipdot-driver-rescue-flipdot-driver-rescue C7
+L flipdot-driver-rescue:C-controller-cache-flipdot-driver-rescue-flipdot-driver-rescue-flipdot-driver-rescue C7
 U 1 1 5C98C550
 P 8300 6700
@@
 $EndComp
 $Comp
-L flipdot-driver-rescue:C-controller-cache-flipdot-driver-rescue-flipdot-driver-rescue C8
+L flipdot-driver-rescue:C-controller-cache-flipdot-driver-rescue-flipdot-driver-rescue-flipdot-driver-rescue C8
 U 1 1 5C98C5EC
 P 8600 6700
@@
 $EndComp
 $Comp
-L flipdot-driver-rescue:C-controller-cache-flipdot-driver-rescue-flipdot-driver-rescue C9
+L flipdot-driver-rescue:C-controller-cache-flipdot-driver-rescue-flipdot-driver-rescue-flipdot-driver-rescue C9
 U 1 1 5CA62C8B
 P 6550 1150
@@
 $EndComp
 $Comp
-L flipdot-driver-rescue:C-controller-cache-flipdot-driver-rescue-flipdot-driver-rescue C11
+L flipdot-driver-rescue:C-controller-cache-flipdot-driver-rescue-flipdot-driver-rescue-flipdot-driver-rescue C11
 U 1 1 5CA62D35
 P 7600 1150
@@
 $EndComp
 $Comp
-L flipdot-driver-rescue:C-controller-cache-flipdot-driver-rescue-flipdot-driver-rescue C12
+L flipdot-driver-rescue:C-controller-cache-flipdot-driver-rescue-flipdot-driver-rescue-flipdot-driver-rescue C12
 U 1 1 5CC51283
 P 7600 4250
@@
 $EndComp
 $Comp
-L flipdot-driver-rescue:C-controller-cache-flipdot-driver-rescue-flipdot-driver-rescue C13
+L flipdot-driver-rescue:C-controller-cache-flipdot-driver-rescue-flipdot-driver-rescue-flipdot-driver-rescue C13
 U 1 1 5CC5134B
 P 7900 4250
@@
 	7150 6200 7150 6100
 $Comp
-L flipdot-driver-rescue:C-controller-cache-flipdot-driver-rescue-flipdot-driver-rescue C10
+L flipdot-driver-rescue:C-controller-cache-flipdot-driver-rescue-flipdot-driver-rescue-flipdot-driver-rescue C10
 U 1 1 5D06CD87
 P 7350 6350
@@
 USART_RX
 $Comp
-L flipdot-driver-rescue:D_Schottky-controller-cache-flipdot-driver-rescue-flipdot-driver-rescue D6
+L flipdot-driver-rescue:D_Schottky-controller-cache-flipdot-driver-rescue-flipdot-driver-rescue-flipdot-driver-rescue D6
 U 1 1 5C783BF6
 P 8700 1150
@@
 $EndComp
 $Comp
-L flipdot-driver-rescue:R-controller-cache-flipdot-driver-rescue-flipdot-driver-rescue R36
+L flipdot-driver-rescue:R-controller-cache-flipdot-driver-rescue-flipdot-driver-rescue-flipdot-driver-rescue R36
 U 1 1 5C29AE4A
 P 7200 2150
@@
 	15000 2350 15500 2350
 $Comp
-L flipdot-driver-rescue:stm32_STM32F103C(8-B)Tx-STM32_converter-cache-flipdot-driver-rescue-flipdot-driver-rescue U6
+L flipdot-driver-rescue:stm32_STM32F103C(8-B)Tx-STM32_converter-cache-flipdot-driver-rescue-flipdot-driver-rescue-flipdot-driver-rescue U6
 U 1 1 5C4F9114
 P 11600 4150
@@
 $EndComp
 $Comp
-L flipdot-driver-rescue:LED-controller-cache-flipdot-driver-rescue-flipdot-driver-rescue D7
+L flipdot-driver-rescue:LED-controller-cache-flipdot-driver-rescue-flipdot-driver-rescue-flipdot-driver-rescue D7
 U 1 1 5DEBAEF3
 P 5650 4350
@@
 $EndComp
 $Comp
-L flipdot-driver-rescue:LED-controller-cache-flipdot-driver-rescue-flipdot-driver-rescue D8
+L flipdot-driver-rescue:LED-controller-cache-flipdot-driver-rescue-flipdot-driver-rescue-flipdot-driver-rescue D8
 U 1 1 5DF44183
 P 6400 4350
@@
 $EndComp
 $Comp
-L flipdot-driver-rescue:CP-controller-cache-flipdot-driver-rescue-flipdot-driver-rescue C16
+L flipdot-driver-rescue:CP-controller-cache-flipdot-driver-rescue-flipdot-driver-rescue-flipdot-driver-rescue C16
 U 1 1 5CF6C5C2
 P 700 2850
@@
 $EndComp
 $Comp
-L flipdot-driver-rescue:C-controller-cache-flipdot-driver-rescue-flipdot-driver-rescue C17
+L flipdot-driver-rescue:C-controller-cache-flipdot-driver-rescue-flipdot-driver-rescue-flipdot-driver-rescue C17
 U 1 1 5CF6CCDF
 P 1050 3000
@@
 $EndComp
 $Comp
-L flipdot-driver-rescue:L-controller-cache-flipdot-driver-rescue-flipdot-driver-rescue L2
+L flipdot-driver-rescue:L-controller-cache-flipdot-driver-rescue-flipdot-driver-rescue-flipdot-driver-rescue L2
 U 1 1 5CF6D440
 P 2600 2350
@@
 $EndComp
 $Comp
-L flipdot-driver-rescue:D_Schottky-controller-cache-flipdot-driver-rescue-flipdot-driver-rescue D2
+L flipdot-driver-rescue:D_Schottky-controller-cache-flipdot-driver-rescue-flipdot-driver-rescue-flipdot-driver-rescue D2
 U 1 1 5CF6DC84
 P 3400 2350
@@
 $EndComp
 $Comp
-L flipdot-driver-rescue:C-controller-cache-flipdot-driver-rescue-flipdot-driver-rescue C20
+L flipdot-driver-rescue:C-controller-cache-flipdot-driver-rescue-flipdot-driver-rescue-flipdot-driver-rescue C20
 U 1 1 5CF6F069
 P 4050 2800
@@
 $EndComp
 $Comp
-L flipdot-driver-rescue:CP-controller-cache-flipdot-driver-rescue-flipdot-driver-rescue C21
+L flipdot-driver-rescue:CP-controller-cache-flipdot-driver-rescue-flipdot-driver-rescue-flipdot-driver-rescue C21
 U 1 1 5CF6F72F
 P 4400 2800
@@
 24V_EN
 $Comp
-L flipdot-driver-rescue:C-controller-cache-flipdot-driver-rescue-flipdot-driver-rescue C19
+L flipdot-driver-rescue:C-controller-cache-flipdot-driver-rescue-flipdot-driver-rescue-flipdot-driver-rescue C19
 U 1 1 5CF703D9
 P 1950 3250
@@
 	800  2550 1050 2550
 $Comp
-L flipdot-driver-rescue:C-controller-cache-flipdot-driver-rescue-flipdot-driver-rescue C18
+L flipdot-driver-rescue:C-controller-cache-flipdot-driver-rescue-flipdot-driver-rescue-flipdot-driver-rescue C18
 U 1 1 5D79E9FF
 P 1350 2850
@@
 Connection ~ 1650 2850
 $Comp
-L flipdot-driver-rescue:AX5201-LCSC-flipdot-driver-rescue U8
+L flipdot-driver-rescue:AX5201-LCSC-flipdot-driver-rescue-flipdot-driver-rescue U8
 U 1 1 5DB4EC83
 P 2600 2950
@@
 USB2_N
 $Comp
-L flipdot-driver-rescue:C-controller-cache-flipdot-driver-rescue-flipdot-driver-rescue C22
+L flipdot-driver-rescue:C-controller-cache-flipdot-driver-rescue-flipdot-driver-rescue-flipdot-driver-rescue C22
 U 1 1 5D0FB237
 P 900 6900
@@
 	900  7050 900  7150
 $Comp
-L flipdot-driver-rescue:R-controller-cache R11
+L flipdot-driver-rescue:R-controller-cache-flipdot-driver-rescue R11
 U 1 1 5D210FC0
 P 4300 5600
@@
 $EndComp
 $Comp
-L flipdot-driver-rescue:R-controller-cache R12
+L flipdot-driver-rescue:R-controller-cache-flipdot-driver-rescue R12
 U 1 1 5D2115E1
 P 4550 5700
@@
 	3700 5700 4150 5700
 $Comp
-L flipdot-driver-rescue:CP-controller-cache-flipdot-driver-rescue-flipdot-driver-rescue C23
+L flipdot-driver-rescue:CP-controller-cache-flipdot-driver-rescue-flipdot-driver-rescue-flipdot-driver-rescue C23
 U 1 1 5D3FC10B
 P 4800 2800
@@
 Wire Wire Line
 	5150 1200 5150 1750
+Wire Wire Line
+	1300 6000 1800 6000
+Wire Wire Line
+	1450 6100 1800 6100
+Wire Wire Line
+	1450 6200 1800 6200
+Wire Wire Line
+	1450 6300 1800 6300
+$Comp
+L Mechanical:Fiducial FID1
+U 1 1 5CFAE734
+P 3700 900
+F 0 "FID1" H 3785 946 50  0000 L CNN
+F 1 "Fiducial" H 3785 855 50  0000 L CNN
+F 2 "Fiducial:Fiducial_0.75mm_Dia_1.5mm_Outer" H 3700 900 50  0001 C CNN
+F 3 "~" H 3700 900 50  0001 C CNN
+	1    3700 900
+	1    0    0    -1
+$EndComp
+$Comp
+L Mechanical:Fiducial FID2
+U 1 1 5CFB7365
+P 3700 1150
+F 0 "FID2" H 3785 1196 50  0000 L CNN
+F 1 "Fiducial" H 3785 1105 50  0000 L CNN
+F 2 "Fiducial:Fiducial_0.75mm_Dia_1.5mm_Outer" H 3700 1150 50  0001 C CNN
+F 3 "~" H 3700 1150 50  0001 C CNN
+	1    3700 1150
+	1    0    0    -1
+$EndComp
+$Comp
+L Mechanical:Fiducial FID3
+U 1 1 5CFB78CB
+P 3700 1400
+F 0 "FID3" H 3785 1446 50  0000 L CNN
+F 1 "Fiducial" H 3785 1355 50  0000 L CNN
+F 2 "Fiducial:Fiducial_0.75mm_Dia_1.5mm_Outer" H 3700 1400 50  0001 C CNN
+F 3 "~" H 3700 1400 50  0001 C CNN
+	1    3700 1400
+	1    0    0    -1
+$EndComp
 $EndSCHEMATC
